File: Talha/schematic/untitled.sch (EAGLE design)
At the start: 4 parts, among them J1 RASPBERRYPI-40-PIN-GPIO_PTH

Commit message: pcb update
Connections:
- removed net N$2: J1.GND@39, J2.7
- net GND: now also J1.GND@39, J2.7
Changed lines of the file:
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@@
 <junction x="-38.1" y="7.62"/>
+</segment>
+<segment>
+<pinref part="J2" gate="G$1" pin="7"/>
+<wire x1="91.44" y1="58.42" x2="86.36" y2="58.42" width="0.1524" layer="91"/>
+<label x="83.82" y="58.42" size="1.778" layer="95"/>
+<wire x1="86.36" y1="17.78" x2="33.02" y2="17.78" width="0.1524" layer="91"/>
+<wire x1="33.02" y1="17.78" x2="30.48" y2="20.32" width="0.1524" layer="91"/>
+<wire x1="30.48" y1="20.32" x2="30.48" y2="27.94" width="0.1524" layer="91"/>
+<pinref part="J1" gate="G$1" pin="GND@39"/>
+<wire x1="30.48" y1="27.94" x2="35.56" y2="27.94" width="0.1524" layer="91"/>
+<wire x1="86.36" y1="17.78" x2="86.36" y2="58.42" width="0.1524" layer="91"/>
 </segment>
 </net>
@@
 </segment>
 </net>
-<net name="N$2" class="0">
-<segment>
-<pinref part="J2" gate="G$1" pin="7"/>
-<wire x1="91.44" y1="58.42" x2="86.36" y2="53.34" width="0.1524" layer="91"/>
-<wire x1="86.36" y1="53.34" x2="86.36" y2="17.78" width="0.1524" layer="91"/>
-<wire x1="86.36" y1="17.78" x2="33.02" y2="17.78" width="0.1524" layer="91"/>
-<wire x1="33.02" y1="17.78" x2="30.48" y2="20.32" width="0.1524" layer="91"/>
-<wire x1="30.48" y1="20.32" x2="30.48" y2="27.94" width="0.1524" layer="91"/>
-<pinref part="J1" gate="G$1" pin="GND@39"/>
-<wire x1="30.48" y1="27.94" x2="35.56" y2="27.94" width="0.1524" layer="91"/>
-</segment>
-</net>
