File: Talha/schematic/untitled.brd (EAGLE design)
At the start: 70 x 51 mm, 4 parts, among them J1 RASPBERRYPI-40-PIN-GPIO_PTH

Commit message: pcb design update
Parts:
- added U$2: (no value), logo:BIOHAZARD_10.00
- added U$3: (no value), logo:EAGLE-PLC-10MM
- added U$4: (no value), logo:RADIOACTIVE_10.00
- added U$5: (no value), logo:TONNE
Routing:
- net VCC: track 79.7 -> 108.0 mm
- net N$1: track 41.8 -> 57.3 mm
- net RX: track 22.4 -> 20.0 mm
- net TX: track 13.1 -> 11.3 mm
- net N$4: track 41.0 -> 42.3 mm
Other:
- board text added: "5V"

Commit message: pcb gerber files generated
Parts:
- removed U$2: (no value), logo:BIOHAZARD_10.00
- renumbered U$1 to XBEE
Changed lines of the file:
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@@
 <drawing>
 <settings>
-<setting alwaysvectorfont="no"/>
+<setting alwaysvectorfont="yes"/>
 <setting verticaltext="up"/>
 </settings>
@@
 <plain>
 <wire x1="19.05" y1="36.83" x2="18.542" y2="36.83" width="0.1524" layer="21"/>
-<text x="10.668" y="32.766" size="1.27" layer="21" ratio="15" rot="R270">VIN</text>
-<text x="28.448" y="32.766" size="1.27" layer="21" ratio="15" rot="R270">3.3V</text>
-<text x="13.462" y="32.766" size="1.27" layer="21" ratio="15" rot="R270">GND</text>
-<text x="23.368" y="32.766" size="1.0668" layer="21" ratio="15" rot="R270">VBAT</text>
-<text x="18.288" y="32.766" size="1.27" layer="21" ratio="15" rot="R270">TX</text>
-<text x="15.748" y="32.766" size="1.27" layer="21" ratio="15" rot="R270">RX</text>
-<text x="25.908" y="32.766" size="1.27" layer="21" ratio="15" rot="R270">EN</text>
-<text x="20.828" y="32.766" size="1.27" layer="21" ratio="15" rot="R270">FIX</text>
-<text x="7.874" y="32.766" size="1.27" layer="21" ratio="15" rot="R270">PPS</text>
+<text x="10.668" y="32.766" size="0.8128" layer="21" rot="R270">VIN</text>
+<text x="28.575" y="32.9438" size="0.8128" layer="21" rot="R270">3.3V</text>
+<text x="13.462" y="32.766" size="0.8128" layer="21" rot="R270">GND</text>
+<text x="23.368" y="32.766" size="0.8128" layer="21" rot="R270">VBAT</text>
+<text x="18.288" y="32.766" size="0.8128" layer="21" rot="R270">TX</text>
+<text x="15.748" y="32.766" size="0.8128" layer="21" rot="R270">RX</text>
+<text x="25.908" y="32.766" size="0.8128" layer="21" rot="R270">EN</text>
+<text x="20.828" y="32.766" size="0.8128" layer="21" rot="R270">FIX</text>
+<text x="7.874" y="32.766" size="0.8128" layer="21" rot="R270">PPS</text>
 <wire x1="8.128" y1="3.048" x2="6.096" y2="5.08" width="0.1524" layer="21" curve="-90"/>
 <wire x1="6.096" y1="5.08" x2="6.096" y2="34.29" width="0.1524" layer="21"/>
@@
 <wire x1="31.496" y1="5.842" x2="28.702" y2="3.048" width="0.1524" layer="21" curve="-90"/>
 <wire x1="28.702" y1="3.048" x2="7.874" y2="3.048" width="0.1524" layer="21"/>
-<text x="43.942" y="17.526" size="1.27" layer="21" ratio="15" rot="R270">3.3V</text>
-<text x="61.976" y="17.526" size="1.27" layer="21" ratio="15" rot="R270">GND</text>
-<text x="45.72" y="18.796" size="1.27" layer="21" ratio="15" rot="R270">DOUT</text>
-<text x="47.752" y="16.764" size="1.27" layer="21" ratio="15" rot="R270">DIN</text>
-<text x="50.8508" y="3.9116" size="1.27" layer="21" ratio="15" rot="R270">3.3V</text>
-<text x="55.88" y="3.81" size="1.27" layer="21" ratio="15" rot="R270">TX</text>
-<text x="58.42" y="3.81" size="1.27" layer="21" ratio="15" rot="R270">RX</text>
-<text x="68.1228" y="6.7056" size="1.397" layer="21" rot="R90">UoR Road Roughness Measurement System</text>
-<text x="53.34" y="4.064" size="1.27" layer="21" ratio="15" rot="R270">GND</text>
+<text x="44.0436" y="16.1036" size="0.8128" layer="21" rot="R270">3.3V</text>
+<text x="62.1792" y="16.4338" size="0.8128" layer="21" rot="R270">GND</text>
+<text x="46.1264" y="17.018" size="0.8128" layer="21" rot="R270">DOUT</text>
+<text x="48.1838" y="15.7988" size="0.8128" layer="21" rot="R270">DIN</text>
+<text x="50.8508" y="3.9116" size="0.8128" layer="21" rot="R270">3.3V</text>
+<text x="55.88" y="3.81" size="0.8128" layer="21" rot="R270">TX</text>
+<text x="58.42" y="3.81" size="0.8128" layer="21" rot="R270">RX</text>
+<text x="67.9704" y="5.1308" size="1.397" layer="21" rot="R90">UoR Road Roughness Measurement System</text>
+<text x="53.34" y="4.064" size="0.8128" layer="21" rot="R270">GND</text>
 <wire x1="0" y1="0" x2="70" y2="0" width="0.1524" layer="20"/>
 <wire x1="70" y1="0" x2="70" y2="51" width="0.1524" layer="20"/>
@@
 <dimension x1="2.54" y1="2.54" x2="67.31" y2="2.54" x3="34.925" y3="-7.62" textsize="1.778" layer="47"/>
 <dimension x1="0" y1="0" x2="70" y2="0" x3="35" y3="-12.7" textsize="1.778" layer="47"/>
-<text x="59.8932" y="45.0596" size="1.27" layer="21" ratio="15">3.3V</text>
-<text x="59.944" y="41.148" size="1.27" layer="21" ratio="15">5V</text>
+<text x="60.6298" y="45.1866" size="0.8128" layer="21">3.3V</text>
+<text x="60.7314" y="41.148" size="0.8128" layer="21">5V</text>
 </plain>
 <attributes>
@@
 </class>
 </classes>
-<designrules name="default">
+<designrules name="default *">
 <description language="de">&lt;b&gt;EAGLE Design Rules&lt;/b&gt;
 &lt;p&gt;
@@
 <param name="layerSetup" value="(1*16)"/>
 <param name="mtCopper" value="0.035mm 0.035mm 0.035mm 0.035mm 0.035mm 0.035mm 0.035mm 0.035mm 0.035mm 0.035mm 0.035mm 0.035mm 0.035mm 0.035mm 0.035mm 0.035mm"/>
-<param name="mtIsolate" value="1.5mm 0.15mm 0.2mm 0.15mm 0.2mm 0.15mm 0.2mm 0.15mm 0.2mm 0.15mm 0.2mm 0.15mm 0.2mm 0.15mm 0.2mm"/>
+<param name="mtIsolate" value="1.53mm 0.15mm 0.2mm 0.15mm 0.2mm 0.15mm 0.2mm 0.15mm 0.2mm 0.15mm 0.2mm 0.15mm 0.2mm 0.15mm 0.2mm"/>
 <param name="mdWireWire" value="6mil"/>
 <param name="mdWirePad" value="6mil"/>
@@
 </element>
 <element name="J2" library="SparkFun-Connectors" library_urn="urn:adsk.eagle:library:513" package="1X09_NO_SILK" package3d_urn="urn:adsk.eagle:package:38156/1" value="" x="28.956" y="35.56" rot="R180"/>
-<element name="U$1" library="adafruit" library_urn="urn:adsk.eagle:library:420" package="XBEE" package3d_urn="urn:adsk.eagle:package:6240840/1" value="XBEE" x="50.038" y="23.368" rot="R90"/>
+<element name="XBEE" library="adafruit" library_urn="urn:adsk.eagle:library:420" package="XBEE" package3d_urn="urn:adsk.eagle:package:6240840/1" value="XBEE" x="50.038" y="23.368" rot="R90"/>
 <element name="J3" library="SparkFun-Connectors" library_urn="urn:adsk.eagle:library:513" package="1X04" package3d_urn="urn:adsk.eagle:package:38085/1" value="" x="58.928" y="5.842" rot="R180">
 <attribute name="PROD_ID" value="CONN-09696" x="58.928" y="5.842" size="1.778" layer="27" rot="R180" display="off"/>
 </element>
-<element name="U$2" library="logo" library_urn="urn:adsk.eagle:library:264" package="BIOHAZARD_10.00" value="" x="7.0358" y="3.9624"/>
 <element name="U$3" library="logo" library_urn="urn:adsk.eagle:library:264" package="EAGLE-PLC-10MM" value="" x="13.9446" y="14.1224"/>
 <element name="U$4" library="logo" library_urn="urn:adsk.eagle:library:264" package="RADIOACTIVE_10.00" value="" x="46.8122" y="20.1676"/>
@@
 <contactref element="J1" pad="6"/>
 <contactref element="J3" pad="3"/>
-<contactref element="U$1" pad="10"/>
+<contactref element="XBEE" pad="10"/>
 <contactref element="J1" pad="34"/>
 <polygon width="0.1524" layer="1" spacing="2.54" isolate="0.4064">
@@
 <signal name="TX">
 <contactref element="J3" pad="2"/>
-<contactref element="U$1" pad="3"/>
+<contactref element="XBEE" pad="3"/>
 <wire x1="56.388" y1="5.842" x2="53.34" y2="8.89" width="0.254" layer="16"/>
 <wire x1="53.34" y1="8.89" x2="50.8" y2="8.89" width="0.254" layer="16"/>
@@
 <signal name="RX">
 <contactref element="J3" pad="1"/>
-<contactref element="U$1" pad="2"/>
+<contactref element="XBEE" pad="2"/>
 <wire x1="58.928" y1="5.842" x2="56.896" y2="3.81" width="0.254" layer="16"/>
 <wire x1="56.896" y1="3.81" x2="49.53" y2="3.81" width="0.254" layer="16"/>
@@
 </signal>
 <signal name="VCC">
-<contactref element="U$1" pad="1"/>
+<contactref element="XBEE" pad="1"/>
 <contactref element="J1" pad="17"/>
 <wire x1="44.538" y1="12.368" x2="42.936" y2="13.97" width="0.508" layer="16"/>

Commit message: complete project folder update
Parts:
- renumbered J1 to ., J2 to GPS_HEADER, J3 to UART
Routing:
- net VCC: track 108.0 -> 0.00 mm
Changed lines of the file:
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@@
 <?xml version="1.0" encoding="utf-8"?>
 <!DOCTYPE eagle SYSTEM "eagle.dtd">
-<eagle version="9.0.0">
+<eagle version="9.3.0">
 <drawing>
 <settings>
-<setting alwaysvectorfont="yes"/>
+<setting alwaysvectorfont="no"/>
 <setting verticaltext="up"/>
 </settings>
@@
 <param name="checkStop" value="0"/>
 <param name="checkValues" value="0"/>
+<param name="checkNames" value="1"/>
+<param name="checkWireStubs" value="1"/>
+<param name="checkPolygonWidth" value="0"/>
 <param name="useDiameter" value="13"/>
 <param name="maxErrors" value="50"/>
@@
 </autorouter>
 <elements>
-<element name="J1" library="SparkFun-Connectors" library_urn="urn:adsk.eagle:library:513" package="2X20_SHROUDED" package3d_urn="urn:adsk.eagle:package:38279/1" value="RASPBERRYPI-40-PIN-GPIO_PTH" x="34.798" y="43.942" rot="R270">
+<element name="." library="SparkFun-Connectors" library_urn="urn:adsk.eagle:library:513" package="2X20_SHROUDED" package3d_urn="urn:adsk.eagle:package:38279/1" value="RASPBERRYPI-40-PIN-GPIO_PTH" x="34.798" y="43.942" smashed="yes" rot="R270">
+<attribute name="NAME" x="64.262" y="48.387" size="0.6096" layer="25" font="vector" ratio="20" rot="R270"/>
 <attribute name="PROD_ID" value="CONN-12263" x="34.798" y="43.942" size="1.778" layer="27" rot="R270" display="off"/>
 <attribute name="SF_ID" value="PRT-13054" x="34.798" y="43.942" size="1.778" layer="27" rot="R270" display="off"/>
+<attribute name="VALUE" x="4.699" y="48.26" size="0.6096" layer="27" font="vector" ratio="20" rot="R270"/>
 </element>
-<element name="J2" library="SparkFun-Connectors" library_urn="urn:adsk.eagle:library:513" package="1X09_NO_SILK" package3d_urn="urn:adsk.eagle:package:38156/1" value="" x="28.956" y="35.56" rot="R180"/>
-<element name="XBEE" library="adafruit" library_urn="urn:adsk.eagle:library:420" package="XBEE" package3d_urn="urn:adsk.eagle:package:6240840/1" value="XBEE" x="50.038" y="23.368" rot="R90"/>
-<element name="J3" library="SparkFun-Connectors" library_urn="urn:adsk.eagle:library:513" package="1X04" package3d_urn="urn:adsk.eagle:package:38085/1" value="" x="58.928" y="5.842" rot="R180">
+<element name="GPS_HEADER" library="SparkFun-Connectors" library_urn="urn:adsk.eagle:library:513" package="1X09_NO_SILK" package3d_urn="urn:adsk.eagle:package:38156/1" value="" x="28.956" y="35.56" smashed="yes" rot="R180">
+<attribute name="NAME" x="30.226" y="34.163" size="0.6096" layer="25" font="vector" ratio="20" rot="R180"/>
+<attribute name="VALUE" x="30.226" y="37.592" size="0.6096" layer="27" font="vector" ratio="20" rot="R180"/>
+</element>
+<element name="XBEE" library="adafruit" library_urn="urn:adsk.eagle:library:420" package="XBEE" package3d_urn="urn:adsk.eagle:package:6240840/1" value="XBEE" x="50.038" y="23.368" smashed="yes" rot="R90">
+<attribute name="NAME" x="66.038" y="20.368" size="1.27" layer="25" rot="R90"/>
+</element>
+<element name="UART" library="SparkFun-Connectors" library_urn="urn:adsk.eagle:library:513" package="1X04" package3d_urn="urn:adsk.eagle:package:38085/1" value="" x="58.928" y="5.842" smashed="yes" rot="R180">
+<attribute name="NAME" x="60.198" y="4.445" size="0.6096" layer="25" font="vector" ratio="20" rot="R180"/>
 <attribute name="PROD_ID" value="CONN-09696" x="58.928" y="5.842" size="1.778" layer="27" rot="R180" display="off"/>
+<attribute name="VALUE" x="60.198" y="7.874" size="0.6096" layer="27" font="vector" ratio="20" rot="R180"/>
 </element>
-<element name="U$3" library="logo" library_urn="urn:adsk.eagle:library:264" package="EAGLE-PLC-10MM" value="" x="13.9446" y="14.1224"/>
-<element name="U$4" library="logo" library_urn="urn:adsk.eagle:library:264" package="RADIOACTIVE_10.00" value="" x="46.8122" y="20.1676"/>
-<element name="U$5" library="logo" library_urn="urn:adsk.eagle:library:264" package="TONNE" value="" x="37.0078" y="5.6642"/>
+<element name="U$3" library="logo" library_urn="urn:adsk.eagle:library:264" package="EAGLE-PLC-10MM" value="" x="13.9446" y="14.1224" smashed="yes"/>
+<element name="U$4" library="logo" library_urn="urn:adsk.eagle:library:264" package="RADIOACTIVE_10.00" value="" x="46.8122" y="20.1676" smashed="yes"/>
+<element name="U$5" library="logo" library_urn="urn:adsk.eagle:library:264" package="TONNE" value="" x="37.0078" y="5.6642" smashed="yes"/>
 </elements>
 <signals>
 <signal name="GND">
-<contactref element="J1" pad="9"/>
-<contactref element="J1" pad="25"/>
-<contactref element="J1" pad="20"/>
-<contactref element="J1" pad="14"/>
-<contactref element="J1" pad="30"/>
-<contactref element="J1" pad="6"/>
-<contactref element="J3" pad="3"/>
+<contactref element="." pad="25"/>
+<contactref element="." pad="20"/>
+<contactref element="." pad="14"/>
+<contactref element="." pad="30"/>
+<contactref element="." pad="6"/>
+<contactref element="UART" pad="3"/>
 <contactref element="XBEE" pad="10"/>
-<contactref element="J1" pad="34"/>
+<contactref element="." pad="34"/>
 <polygon width="0.1524" layer="1" spacing="2.54" isolate="0.4064">
 <vertex x="0" y="51"/>
@@
 <vertex x="0" y="0"/>
 </polygon>
-<contactref element="J2" pad="7"/>
-<contactref element="J1" pad="39"/>
+<contactref element="GPS_HEADER" pad="7"/>
+<contactref element="." pad="9"/>
+<contactref element="." pad="39"/>
+<wire x1="48.768" y1="45.212" x2="53.848" y2="42.672" width="0" layer="19" extent="1-1"/>
+<wire x1="43.688" y1="42.672" x2="48.768" y2="45.212" width="0" layer="19" extent="1-1"/>
+<wire x1="36.068" y1="42.672" x2="43.688" y2="42.672" width="0" layer="19" extent="1-1"/>
+<wire x1="28.448" y1="45.212" x2="36.068" y2="42.672" width="0" layer="19" extent="1-1"/>
+<wire x1="23.368" y1="42.672" x2="28.448" y2="45.212" width="0" layer="19" extent="1-1"/>
+<wire x1="18.288" y1="42.672" x2="23.368" y2="42.672" width="0" layer="19" extent="1-1"/>
+<wire x1="10.668" y1="45.212" x2="18.288" y2="42.672" width="0" layer="19" extent="1-1"/>
+<wire x1="13.716" y1="35.56" x2="18.288" y2="42.672" width="0" layer="19" extent="1-1"/>
+<wire x1="62.538" y1="12.368" x2="53.848" y2="42.672" width="0" layer="19" extent="1-1"/>
+<wire x1="53.848" y1="5.842" x2="62.538" y2="12.368" width="0" layer="19" extent="1-1"/>
 </signal>
 <signal name="5V">
-<contactref element="J1" pad="4"/>
-<contactref element="J1" pad="2"/>
+<contactref element="." pad="4"/>
+<contactref element="." pad="2"/>
 <wire x1="58.928" y1="42.672" x2="56.388" y2="42.672" width="0.508" layer="16"/>
 </signal>
 <signal name="TX">
-<contactref element="J3" pad="2"/>
+<contactref element="UART" pad="2"/>
 <contactref element="XBEE" pad="3"/>
 <wire x1="56.388" y1="5.842" x2="53.34" y2="8.89" width="0.254" layer="16"/>
@@
 </signal>
 <signal name="RX">
-<contactref element="J3" pad="1"/>
+<contactref element="UART" pad="1"/>
 <contactref element="XBEE" pad="2"/>
 <wire x1="58.928" y1="5.842" x2="56.896" y2="3.81" width="0.254" layer="16"/>
@@
 <wire x1="46.538" y1="6.802" x2="46.538" y2="12.368" width="0.254" layer="16"/>
 </signal>
-<signal name="VCC">
-<contactref element="XBEE" pad="1"/>
-<contactref element="J1" pad="17"/>
-<wire x1="44.538" y1="12.368" x2="42.936" y2="13.97" width="0.508" layer="16"/>
-<wire x1="3.81" y1="16.51" x2="6.35" y2="13.97" width="0.508" layer="16"/>
-<wire x1="42.936" y1="13.97" x2="6.35" y2="13.97" width="0.508" layer="16"/>
-<wire x1="7.62" y1="48.26" x2="35.56" y2="48.26" width="0.508" layer="16"/>
-<wire x1="35.56" y1="48.26" x2="38.608" y2="45.212" width="0.508" layer="16"/>
-<wire x1="3.81" y1="16.51" x2="3.81" y2="44.45" width="0.508" layer="16"/>
-<wire x1="3.81" y1="44.45" x2="7.62" y2="48.26" width="0.508" layer="16"/>
-</signal>
 <signal name="N$1">
-<contactref element="J1" pad="1"/>
-<contactref element="J2" pad="1"/>
+<contactref element="." pad="1"/>
+<contactref element="GPS_HEADER" pad="1"/>
 <wire x1="28.956" y1="35.56" x2="36.83" y2="35.56" width="0.508" layer="16"/>
 <wire x1="64.77" y1="31.75" x2="66.04" y2="33.02" width="0.508" layer="16"/>
@@
 </signal>
 <signal name="N$4">
-<contactref element="J1" pad="8"/>
-<contactref element="J2" pad="6"/>
+<contactref element="." pad="8"/>
+<contactref element="GPS_HEADER" pad="6"/>
 <wire x1="20.1168" y1="36.0650125" x2="20.8309875" y2="36.7792" width="0.254" layer="16"/>
 <wire x1="38.0492" y1="36.7792" x2="38.1" y2="36.83" width="0.254" layer="16"/>
@@
 </signal>
 <signal name="N$3">
-<contactref element="J1" pad="10"/>
-<contactref element="J2" pad="5"/>
+<contactref element="." pad="10"/>
+<contactref element="GPS_HEADER" pad="5"/>
 <wire x1="18.796" y1="35.56" x2="21.336" y2="38.1" width="0.254" layer="16"/>
 <wire x1="48.768" y1="39.878" x2="48.768" y2="42.672" width="0.254" layer="16"/>
@@
 <via x="2.54" y="2.54" extent="1-16" drill="2.2" shape="square"/>
 </signal>
+<signal name="VCC">
+<contactref element="XBEE" pad="1"/>
+<contactref element="." pad="17"/>
+<wire x1="44.538" y1="12.368" x2="38.608" y2="45.212" width="0" layer="19" extent="1-1"/>
+</signal>
 </signals>
+<mfgpreviewcolors>
+<mfgpreviewcolor name="soldermaskcolor" color="0xC8008000"/>
+<mfgpreviewcolor name="silkscreencolor" color="0xFFFEFEFE"/>
+<mfgpreviewcolor name="backgroundcolor" color="0xFF282828"/>
+<mfgpreviewcolor name="coppercolor" color="0xFFFFBF00"/>
+<mfgpreviewcolor name="substratecolor" color="0xFF786E46"/>
+</mfgpreviewcolors>
 </board>
 </drawing>
