File: Natnael/schematic/New_Project/ACC.brd (EAGLE design)
At the start: 100 x 100 mm, 10 parts, among them J4 B2B-PH-K-S(LF)(SN)

Commit message: updatae on pcb
Parts:
- J4: value B2B-PH-K-S(LF)(SN) -> 1935161; device B2B-PH-K-S_LF__SN_:JST_B2B-PH-K-S(LF)(SN) -> 1935161:PHOENIX_1935161
- moved J3 12.7 mm to (11.5, 62.3), turned to 270 degrees
- moved J4 2.83 mm to (33.0, 90.2)
- moved J1 1.27 mm to (90.1, 42.2)
Connections:
- net GND: now also J4.1; no longer J4.2
- net N$1: now also J4.2; no longer J4.1
Routing:
- net 3V3: track 250.9 -> 310.6 mm
- net PA2: track 5.52 -> 50.6 mm
- net PA3: track 29.3 -> 49.9 mm
- net PA9: track 44.1 -> 51.9 mm
- net PB6: track 42.8 -> 46.9 mm
- net PB7: track 18.0 -> 20.6 mm
- net N$1: track 11.5 -> 9.47 mm
- net PB5: track 15.9 -> 17.1 mm
- net PA10: track 62.1 -> 61.6 mm

Commit message: pcb design update
Parts:
- added U$1: (no value), logo:BIOHAZARD_10.00
- added U$2: (no value), logo:EAGLE-PLC-8MM
- added U$3: (no value), logo:ESD_10.00
- added U$4: (no value), logo:TONNE
- added U$5: (no value), micro-philips:I2C
- moved J3 2.54 mm to (14.0, 62.3)
- flipped J1 to the top, turned to 180 degrees
- flipped J2 to the top, turned to 180 degrees
Routing:
- net PB7: vias 0 -> 1
- net PB6: vias 0 -> 1
- net PB5: vias 0 -> 1
- net PA9: vias 0 -> 1
- net PA3: vias 0 -> 1
- net PA2: vias 0 -> 1
- net PA10: vias 0 -> 1
- net 3V3: vias 0 -> 1

Commit message: pcb gerber files generated
Parts:
- removed U$1: (no value), logo:BIOHAZARD_10.00
- added U$6: (no value), logo:RADIOACTIVE_10.00
- CIN: value (none) -> 1uF
- COUT: value (none) -> 2.2uF
- moved U$2 77.6 mm to (10.2, 85.1)
- moved U$4 34.4 mm to (55.9, 8.89)
- moved U$3 30.6 mm to (34.3, 7.62)
- moved U$5 2.54 mm to (77.5, 15.2)
- turned XBEE to 270 degrees
- renumbered ACC to MPU6050
Connections:
- removed net 3V3S: J2.4
- removed net N$1: CIN.1, J4.2
- removed net N$2: CIN.2, LP2950.3
- new net VBAT: J2.5
- new net VIN: CIN.1, J4.1, LP2950.3
- net 3V3: now also J2.4; no longer J2.5
- net GND: now also CIN.2, J4.2; no longer J4.1
Routing:
- net 3V3: track 310.6 -> 214.3 mm, vias 1 -> 0
- net PA10: track 61.6 -> 20.1 mm, vias 1 -> 0
- net VIN: track 0.00 -> 33.4 mm
- net PA9: track 51.9 -> 19.2 mm, vias 1 -> 0
- net N$2: track 13.2 -> 0.00 mm
- net N$1: track 9.47 -> 0.00 mm
- net PB6: track 46.9 -> 50.6 mm, vias 1 -> 0
- net PB7: track 20.6 -> 21.5 mm, vias 1 -> 0
- net PA2: track 50.6 -> 49.9 mm, vias 1 -> 0
- net PB5: track 17.1 -> 17.2 mm, vias 1 -> 0
- net PA3: vias 1 -> 0
Other:
- board text added: "VIN"
- board text added: "VOUT"
- board text removed: "JST"

Commit message: complete project folder update
Parts:
- removed U$4: (no value), logo:TONNE
- renumbered LP2950 to VOLTAGE_REGULATOR
Connections:
- new net N$1: MPU6050.8
- new net VCC: XBEE.1
- net 3V3: no longer MPU6050.8, XBEE.1
Routing:
- net 3V3: track 214.3 -> 126.0 mm
- net VCC: track 0.00 -> 74.8 mm
Changed lines of the file:
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@@
 <?xml version="1.0" encoding="utf-8"?>
 <!DOCTYPE eagle SYSTEM "eagle.dtd">
-<eagle version="9.0.0">
+<eagle version="9.3.0">
 <drawing>
 <settings>
-<setting alwaysvectorfont="yes"/>
+<setting alwaysvectorfont="no"/>
 <setting verticaltext="up"/>
 </settings>
@@
 <param name="checkStop" value="0"/>
 <param name="checkValues" value="0"/>
+<param name="checkNames" value="1"/>
+<param name="checkWireStubs" value="1"/>
+<param name="checkPolygonWidth" value="0"/>
 <param name="useDiameter" value="13"/>
 <param name="maxErrors" value="50"/>
@@
 <attribute name="VALUE" x="91.3454" y="44.2374" size="0.6096" layer="27" font="vector" ratio="20" rot="R180"/>
 </element>
-<element name="J2" library="SparkFun-Connectors" library_urn="urn:adsk.eagle:library:513" package="1X29" package3d_urn="urn:adsk.eagle:package:38212/1" value="" x="90.0754" y="72.4154" rot="R180"/>
+<element name="J2" library="SparkFun-Connectors" library_urn="urn:adsk.eagle:library:513" package="1X29" package3d_urn="urn:adsk.eagle:package:38212/1" value="" x="90.0754" y="72.4154" smashed="yes" rot="R180">
+<attribute name="NAME" x="91.3454" y="71.0184" size="0.6096" layer="25" font="vector" ratio="20" rot="R180"/>
+<attribute name="VALUE" x="91.3454" y="74.4474" size="0.6096" layer="27" font="vector" ratio="20" rot="R180"/>
+</element>
 <element name="J3" library="SparkFun-Connectors" library_urn="urn:adsk.eagle:library:513" package="1X06" package3d_urn="urn:adsk.eagle:package:38009/1" value="" x="13.9954" y="62.2554" smashed="yes" rot="R270">
 <attribute name="NAME" x="14.27215625" y="65.135996875" size="0.6096" layer="25" font="vector" ratio="20" rot="R270"/>
@@
 <attribute name="VALUE" x="91.4654" y="85.8774" size="0.6096" layer="27" font="vector" ratio="20" rot="R180"/>
 </element>
-<element name="LP2950" library="linear" library_urn="urn:adsk.eagle:library:262" package="TO92" package3d_urn="urn:adsk.eagle:package:16416/2" value="LP2950Z" x="57.1754" y="91.4654" smashed="yes" rot="R90">
+<element name="VOLTAGE_REGULATOR" library="linear" library_urn="urn:adsk.eagle:library:262" package="TO92" package3d_urn="urn:adsk.eagle:package:16416/2" value="LP2950Z" x="57.1754" y="91.4654" smashed="yes" rot="R90">
 <attribute name="VALUE" x="53.2854" y="89.5564" size="0.8" layer="27" rot="R90"/>
 </element>
@@
 <attribute name="SPICEPREFIX" value="B" x="33.02" y="90.17" size="1.778" layer="27" rot="R90" display="off"/>
 </element>
-<element name="U$2" library="logo" library_urn="urn:adsk.eagle:library:264" package="EAGLE-PLC-8MM" value="" x="10.16" y="85.09"/>
-<element name="U$3" library="logo" library_urn="urn:adsk.eagle:library:264" package="ESD_10.00" value="" x="34.29" y="7.62"/>
-<element name="U$4" library="logo" library_urn="urn:adsk.eagle:library:264" package="TONNE" value="" x="55.88" y="8.89"/>
-<element name="U$5" library="micro-philips" library_urn="urn:adsk.eagle:library:290" package="I2C" value="" x="77.47" y="15.24"/>
-<element name="U$6" library="logo" library_urn="urn:adsk.eagle:library:264" package="RADIOACTIVE_10.00" value="" x="16.47" y="16.86"/>
+<element name="U$2" library="logo" library_urn="urn:adsk.eagle:library:264" package="EAGLE-PLC-8MM" value="" x="10.16" y="85.09" smashed="yes"/>
+<element name="U$3" library="logo" library_urn="urn:adsk.eagle:library:264" package="ESD_10.00" value="" x="34.29" y="7.62" smashed="yes"/>
+<element name="U$5" library="micro-philips" library_urn="urn:adsk.eagle:library:290" package="I2C" value="" x="77.47" y="15.24" smashed="yes">
+<attribute name="NAME" x="80.01" y="15.875" size="0.0254" layer="25"/>
+<attribute name="VALUE" x="80.645" y="15.875" size="0.0254" layer="27"/>
+</element>
+<element name="U$6" library="logo" library_urn="urn:adsk.eagle:library:264" package="RADIOACTIVE_10.00" value="" x="16.47" y="16.86" smashed="yes"/>
 </elements>
 <signals>
@@
 <contactref element="XBEE" pad="10"/>
 <contactref element="J5" pad="1"/>
-<contactref element="LP2950" pad="2"/>
+<contactref element="VOLTAGE_REGULATOR" pad="2"/>
 <contactref element="COUT" pad="2"/>
 <polygon width="0.254" layer="1" isolate="0.3048">
@@
 </signal>
 <signal name="3V3">
-<contactref element="MPU6050" pad="8"/>
-<contactref element="XBEE" pad="1"/>
-<contactref element="LP2950" pad="1"/>
-<contactref element="COUT" pad="1"/>
-<wire x1="88.9254" y1="26.6954" x2="93.98" y2="31.75" width="0.508" layer="16"/>
 <wire x1="93.98" y1="31.75" x2="93.98" y2="57.15" width="0.508" layer="16"/>
-<wire x1="57.1754" y1="90.1954" x2="57.2008" y2="90.17" width="0.508" layer="16"/>
 <wire x1="57.2008" y1="90.17" x2="91.44" y2="90.17" width="0.508" layer="16"/>
 <wire x1="91.44" y1="90.17" x2="93.98" y2="87.63" width="0.508" layer="16"/>
 <wire x1="93.98" y1="78.74" x2="92.71" y2="77.47" width="0.508" layer="16"/>
 <wire x1="93.98" y1="87.63" x2="93.98" y2="78.74" width="0.508" layer="16"/>
-<wire x1="27.1154" y1="31.3454" x2="30.48" y2="27.9808" width="0.508" layer="16"/>
-<wire x1="33.02" y1="16.51" x2="85.09" y2="16.51" width="0.508" layer="16"/>
-<wire x1="88.9254" y1="20.3454" x2="88.9254" y2="26.6954" width="0.508" layer="16"/>
-<wire x1="30.48" y1="27.9808" x2="30.48" y2="19.05" width="0.508" layer="16"/>
-<wire x1="30.48" y1="19.05" x2="33.02" y2="16.51" width="0.508" layer="16"/>
-<wire x1="85.09" y1="16.51" x2="88.9254" y2="20.3454" width="0.508" layer="16"/>
-<wire x1="44.4754" y1="87.6554" x2="44.5008" y2="87.63" width="0.508" layer="16"/>
-<wire x1="44.5008" y1="87.63" x2="54.61" y2="87.63" width="0.508" layer="16"/>
-<wire x1="54.61" y1="87.63" x2="57.1754" y2="90.1954" width="0.508" layer="16"/>
-<wire x1="44.4754" y1="87.6554" x2="44.45" y2="87.63" width="0.508" layer="16"/>
 <contactref element="J2" pad="4"/>
 <wire x1="82.4554" y1="62.3246" x2="82.4554" y2="72.4154" width="0.508" layer="16"/>
@@
 <wire x1="82.4554" y1="76.1054" x2="82.4554" y2="72.4154" width="0.508" layer="16"/>
 <wire x1="83.82" y1="77.47" x2="82.4554" y2="76.1054" width="0.508" layer="16"/>
+<contactref element="VOLTAGE_REGULATOR" pad="1"/>
+<contactref element="COUT" pad="1"/>
+<wire x1="44.4754" y1="87.6554" x2="44.5008" y2="87.63" width="0.508" layer="16"/>
+<wire x1="44.5008" y1="87.63" x2="54.61" y2="87.63" width="0.508" layer="16"/>
+<wire x1="54.61" y1="87.63" x2="57.1754" y2="90.1954" width="0.508" layer="16"/>
+<wire x1="44.4754" y1="87.6554" x2="44.45" y2="87.63" width="0.508" layer="16"/>
+<wire x1="57.2008" y1="90.17" x2="57.1754" y2="90.1954" width="0" layer="19" extent="16-16"/>
 </signal>
 <signal name="NC1">
@@
 </signal>
 <signal name="VIN">
-<contactref element="LP2950" pad="3"/>
+<contactref element="VOLTAGE_REGULATOR" pad="3"/>
 <wire x1="44.45" y1="97.79" x2="41.9354" y2="95.2754" width="0.508" layer="16"/>
 <wire x1="57.1754" y1="96.4946" x2="57.1754" y2="92.7354" width="0.508" layer="16"/>
@@
 <contactref element="J2" pad="5"/>
 </signal>
+<signal name="N$1">
+<contactref element="MPU6050" pad="8"/>
+</signal>
+<signal name="VCC">
+<contactref element="XBEE" pad="1"/>
+<wire x1="27.1154" y1="31.3454" x2="30.48" y2="27.9808" width="0.508" layer="16"/>
+<wire x1="33.02" y1="16.51" x2="85.09" y2="16.51" width="0.508" layer="16"/>
+<wire x1="30.48" y1="27.9808" x2="30.48" y2="19.05" width="0.508" layer="16"/>
+<wire x1="30.48" y1="19.05" x2="33.02" y2="16.51" width="0.508" layer="16"/>
+<wire x1="85.09" y1="16.51" x2="88.9254" y2="20.3454" width="0.508" layer="16"/>
+</signal>
 </signals>
+<mfgpreviewcolors>
+<mfgpreviewcolor name="soldermaskcolor" color="0xC8008000"/>
+<mfgpreviewcolor name="silkscreencolor" color="0xFFFEFEFE"/>
+<mfgpreviewcolor name="backgroundcolor" color="0xFF282828"/>
+<mfgpreviewcolor name="coppercolor" color="0xFFFFBF00"/>
+<mfgpreviewcolor name="substratecolor" color="0xFF786E46"/>
+</mfgpreviewcolors>
 </board>
 </drawing>
